File: KiCad/stepad/stepad.kicad_sch (KiCad schematic)
At the start: 69 parts, among them J1 TYPE-C-31-M12_13_EDITED, J2 Conn_01x03, SW1 MX_Lekker, SW2 MX_Lekker, SW3 MX_Lekker, SW4 MX_Lekker, SW5 SW_Push, SW6 SW_Push, U1 AH49-E, U2 AH49-E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

Commit message: Adding part numbers and updating some footprints
Parts:
- D1, D2, D3, D4: Part Number (none) -> QBLP677R-RGB
- D5, D6: Part Number (none) -> 1N4148W-13-F
- J1: Part Number (none) -> USB4105-GF-A
- SW5, SW6: Part Number (none) -> MSLPT5252AG3TR
- U1, U2, U3, U4: Part Number (none) -> AH49-E
- U5: Part Number (none) -> NCP1117-3.3_SOT223
- U6: Part Number (none) -> W25Q32JVSS
- U7: Part Number (none) -> RP2040
- U8: Part Number (none) -> WE-TVS-82400102
- Y1: footprint Crystal:Crystal_SMD_5032-4Pin_5.0x3.2mm -> Crystal:Crystal_SMD_3225-4Pin_3.2x2.5mm; Part Number (none) -> RH100-12.000-18-2030-TR
Changed lines of the file:
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@@
+      (effects (font (size 1.27 1.27)) hide)
+    )
+    (property "Part Number" "USB4105-GF-A" (id 4) (at 38.1 184.15 0)
       (effects (font (size 1.27 1.27)) hide)
     )
@@
       (effects (font (size 1.27 1.27)) hide)
     )
+    (property "Part Number" "W25Q32JVSS" (id 4) (at 219.71 140.97 0)
+      (effects (font (size 1.27 1.27)) hide)
+    )
     (pin "1")
     (pin "2")
@@
       (effects (font (size 1.27 1.27)) hide)
     )
+    (property "Description" "0.1in pitch pin headers" (id 4) (at 102.87 251.46 0)
+      (effects (font (size 1.27 1.27)) hide)
+    )
     (pin "1")
     (pin "2")
@@
       (effects (font (size 1.27 1.27)) hide)
     )
+    (property "Part Number" "1N4148W-13-F" (id 4) (at 231.14 257.81 0)
+      (effects (font (size 1.27 1.27)) hide)
+    )
     (pin "1")
     (pin "2")
@@
       (effects (font (size 1.27 1.27)) hide)
     )
+    (property "Part Number" "MSLPT5252AG3TR" (id 4) (at 181.61 144.78 0)
+      (effects (font (size 1.27 1.27)) hide)
+    )
     (pin "1")
     (pin "2")
@@
       (effects (font (size 1.27 1.27)) hide)
     )
+    (property "Part Number" "MSLPT5252AG3TR" (id 4) (at 193.04 194.31 0)
+      (effects (font (size 1.27 1.27)) hide)
+    )
     (pin "1")
     (pin "2")
@@
     (property "Reference" "Y1" (id 0) (at 232.41 160.02 90))
     (property "Value" "Crystal_GND24" (id 1) (at 232.41 162.56 90))
-    (property "Footprint" "Crystal:Crystal_SMD_5032-4Pin_5.0x3.2mm" (id 2) (at 227.33 168.91 0)
+    (property "Footprint" "Crystal:Crystal_SMD_3225-4Pin_3.2x2.5mm" (id 2) (at 227.33 168.91 0)
       (effects (font (size 1.27 1.27)) hide)
     )
     (property "Datasheet" "~" (id 3) (at 227.33 168.91 0)
+      (effects (font (size 1.27 1.27)) hide)
+    )
+    (property "Description" "12 MHz Crystal" (id 4) (at 227.33 168.91 0)
+      (effects (font (size 1.27 1.27)) hide)
+    )
+    (property "Part Number" "RH100-12.000-18-2030-TR" (id 5) (at 227.33 168.91 0)
       (effects (font (size 1.27 1.27)) hide)
     )
@@
       (effects (font (size 1.27 1.27)) hide)
     )
+    (property "Part Number" "NCP1117-3.3_SOT223" (id 4) (at 261.62 53.34 0)
+      (effects (font (size 1.27 1.27)) hide)
+    )
     (pin "1")
     (pin "2")
@@
       (effects (font (size 1.27 1.27)) hide)
     )
+    (property "Part Number" "AH49-E" (id 4) (at 107.95 50.8 0)
+      (effects (font (size 1.27 1.27)) hide)
+    )
     (pin "1")
     (pin "2")
@@
       (effects (font (size 1.27 1.27)) hide)
     )
+    (property "Part Number" "1N4148W-13-F" (id 4) (at 219.71 257.81 0)
+      (effects (font (size 1.27 1.27)) hide)
+    )
     (pin "1")
     (pin "2")
@@
     )
     (property "Datasheet" "" (id 3) (at 137.16 50.8 0)
+      (effects (font (size 1.27 1.27)) hide)
+    )
+    (property "Part Number" "AH49-E" (id 4) (at 137.16 50.8 0)
       (effects (font (size 1.27 1.27)) hide)
     )
@@
       (effects (font (size 1.27 1.27)) hide)
     )
+    (property "Part Number" "AH49-E" (id 4) (at 50.8 50.8 0)
+      (effects (font (size 1.27 1.27)) hide)
+    )
     (pin "1")
     (pin "2")
@@
       (effects (font (size 1.27 1.27)) hide)
     )
+    (property "Part Number" "QBLP677R-RGB" (id 4) (at 85.09 113.03 0)
+      (effects (font (size 1.27 1.27)) hide)
+    )
     (pin "1")
     (pin "2")
@@
     )
     (property "Datasheet" "" (id 3) (at 264.16 163.83 0)
+      (effects (font (size 1.27 1.27)) hide)
+    )
+    (property "Part Number" "RP2040" (id 4) (at 283.21 163.83 0)
       (effects (font (size 1.27 1.27)) hide)
     )
@@
       (effects (font (size 1.27 1.27)) hide)
     )
+    (property "Part Number" "QBLP677R-RGB" (id 4) (at 143.51 113.03 0)
+      (effects (font (size 1.27 1.27)) hide)
+    )
     (pin "1")
     (pin "2")
@@
       (effects (font (size 1.27 1.27)) hide)
     )
+    (property "Part Number" "QBLP677R-RGB" (id 4) (at 114.3 113.03 0)
+      (effects (font (size 1.27 1.27)) hide)
+    )
     (pin "1")
     (pin "2")
@@
       (effects (font (size 1.27 1.27)) hide)
     )
+    (property "Part Number" "QBLP677R-RGB" (id 4) (at 57.15 113.03 0)
+      (effects (font (size 1.27 1.27)) hide)
+    )
     (pin "1")
     (pin "2")
@@
     )
     (property "Datasheet" "https://katalog.we-online.de/pbs/datasheet/82400102.pdf" (id 3) (at 81.28 195.58 0)
+      (effects (font (size 1.27 1.27)) hide)
+    )
+    (property "Part Number" "WE-TVS-82400102" (id 4) (at 81.28 189.23 0)
       (effects (font (size 1.27 1.27)) hide)
     )
@@
       (effects (font (size 1.27 1.27)) hide)
     )
+    (property "Part Number" "AH49-E" (id 4) (at 78.74 50.8 0)
+      (effects (font (size 1.27 1.27)) hide)
+    )
     (pin "1")
     (pin "2")
@@
     )
     (path "/6ff83143-7f67-4daf-a16c-8739d670aeaf"
-      (reference "Y1") (unit 1) (value "Crystal_GND24") (footprint "Crystal:Crystal_SMD_5032-4Pin_5.0x3.2mm")
-    )
-  )
+      (reference "Y1") (unit 1) (value "Crystal_GND24") (footprint "Crystal:Crystal_SMD_3225-4Pin_3.2x2.5mm")
+    )
+  )

Commit message: Updating part numbers and gerber files
Parts:
- C1, C10, C11, C12, C13, C14, C15, C16, C17, C18, C2, C21, C24, C3, C4, C5: Part Number (none) -> C0603C104M4RAC7411
- C19, C20: Part Number (none) -> CL10A105KA8NNNC
- C22, C23: Part Number (none) -> C0603C270J3GAC7867
- R1, R2, R3, R4: Part Number (none) -> RC0603FR-070RL
- R11, R16: Part Number (none) -> RNCP0603FTD10K0
- R14, R15: Part Number (none) -> RC0603FR-135K1L
- R5, R6, R7: Part Number (none) -> RC0603JR-07300RL
- R8, R9: Part Number (none) -> RC0603FR-1327RL
Changed lines of the file:
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@@
+      (effects (font (size 1.27 1.27)) hide)
+    )
+    (property "Part Number" "C0603C104M4RAC7411" (id 4) (at 101.6 41.91 0)
       (effects (font (size 1.27 1.27)) hide)
     )
@@
       (effects (font (size 1.27 1.27)) hide)
     )
+    (property "Part Number" "C0603C104M4RAC7411" (id 4) (at 72.39 41.91 0)
+      (effects (font (size 1.27 1.27)) hide)
+    )
     (pin "1")
     (pin "2")
@@
     )
     (property "Datasheet" "~" (id 3) (at 372.11 92.71 0)
+      (effects (font (size 1.27 1.27)) hide)
+    )
+    (property "Part Number" "C0603C104M4RAC7411" (id 4) (at 372.11 92.71 0)
       (effects (font (size 1.27 1.27)) hide)
     )
@@
       (effects (font (size 1.27 1.27)) hide)
     )
+    (property "Part Number" "RC0603FR-070RL" (id 4) (at 54.61 62.23 0)
+      (effects (font (size 1.27 1.27)) hide)
+    )
     (pin "1")
     (pin "2")
@@
     )
     (property "Datasheet" "~" (id 3) (at 314.96 92.71 0)
+      (effects (font (size 1.27 1.27)) hide)
+    )
+    (property "Part Number" "C0603C104M4RAC7411" (id 4) (at 314.96 92.71 0)
       (effects (font (size 1.27 1.27)) hide)
     )
@@
       (effects (font (size 1.27 1.27)) hide)
     )
+    (property "Part Number" "C0603C104M4RAC7411" (id 4) (at 360.68 92.71 0)
+      (effects (font (size 1.27 1.27)) hide)
+    )
     (pin "1")
     (pin "2")
@@
       (effects (font (size 1.27 1.27)) hide)
     )
+    (property "Part Number" "C0603C104M4RAC7411" (id 4) (at 44.45 41.91 0)
+      (effects (font (size 1.27 1.27)) hide)
+    )
     (pin "1")
     (pin "2")
@@
       (effects (font (size 1.27 1.27)) hide)
     )
+    (property "Part Number" "RC0603JR-07300RL" (id 4) (at 43.18 111.76 0)
+      (effects (font (size 1.27 1.27)) hide)
+    )
     (pin "1")
     (pin "2")
@@
       (effects (font (size 1.27 1.27)) hide)
     )
+    (property "Part Number" "C0603C104M4RAC7411" (id 4) (at 199.39 128.27 0)
+      (effects (font (size 1.27 1.27)) hide)
+    )
     (pin "1")
     (pin "2")
@@
     )
     (property "Datasheet" "~" (id 3) (at 337.82 92.71 0)
+      (effects (font (size 1.27 1.27)) hide)
+    )
+    (property "Part Number" "C0603C104M4RAC7411" (id 4) (at 337.82 92.71 0)
       (effects (font (size 1.27 1.27)) hide)
     )
@@
       (effects (font (size 1.27 1.27)) hide)
     )
+    (property "Part Number" "C0603C104M4RAC7411" (id 4) (at 130.81 41.91 0)
+      (effects (font (size 1.27 1.27)) hide)
+    )
     (pin "1")
     (pin "2")
@@
       (effects (font (size 1.27 1.27)) hide)
     )
+    (property "Part Number" "C0603C104M4RAC7411" (id 4) (at 92.71 196.85 0)
+      (effects (font (size 1.27 1.27)) hide)
+    )
     (pin "1")
     (pin "2")
@@
     )
     (property "Datasheet" "~" (id 3) (at 241.3 92.71 0)
+      (effects (font (size 1.27 1.27)) hide)
+    )
+    (property "Part Number" "C0603C104M4RAC7411" (id 4) (at 241.3 92.71 0)
       (effects (font (size 1.27 1.27)) hide)
     )
@@
       (effects (font (size 1.27 1.27)) hide)
     )
+    (property "Part Number" "RC0603FR-135K1L" (id 4) (at 60.96 172.72 0)
+      (effects (font (size 1.27 1.27)) hide)
+    )
     (pin "1")
     (pin "2")
@@
       (effects (font (size 1.27 1.27)) hide)
     )
+    (property "Part Number" "RC0603FR-070RL" (id 4) (at 111.76 62.23 0)
+      (effects (font (size 1.27 1.27)) hide)
+    )
     (pin "1")
     (pin "2")
@@
       (effects (font (size 1.27 1.27)) hide)
     )
+    (property "Part Number" "C0603C270J3GAC7867" (id 4) (at 217.17 172.72 0)
+      (effects (font (size 1.27 1.27)) hide)
+    )
     (pin "1")
     (pin "2")
@@
       (effects (font (size 1.27 1.27)) hide)
     )
+    (property "Part Number" "RC0603FR-070RL" (id 4) (at 82.55 62.23 0)
+      (effects (font (size 1.27 1.27)) hide)
+    )
     (pin "1")
     (pin "2")
@@
       (effects (font (size 1.27 1.27)) hide)
     )
+    (property "Part Number" "C0603C104M4RAC7411" (id 4) (at 326.39 92.71 0)
+      (effects (font (size 1.27 1.27)) hide)
+    )
     (pin "1")
     (pin "2")
@@
       (effects (font (size 1.27 1.27)) hide)
     )
+    (property "Part Number" "RC0603FR-135K1L" (id 4) (at 60.96 167.64 0)
+      (effects (font (size 1.27 1.27)) hide)
+    )
     (pin "1")
     (pin "2")
@@
       (effects (font (size 1.27 1.27)) hide)
     )
+    (property "Part Number" "RC0603FR-1327RL" (id 4) (at 322.58 120.65 0)
+      (effects (font (size 1.27 1.27)) hide)
+    )
     (pin "1")
     (pin "2")
@@
       (effects (font (size 1.27 1.27)) hide)
     )
+    (property "Part Number" "RNCP0603FTD10K0" (id 4) (at 182.88 184.15 0)
+      (effects (font (size 1.27 1.27)) hide)
+    )
     (pin "1")
     (pin "2")
@@
     )
     (property "Datasheet" "~" (id 3) (at 349.25 92.71 0)
+      (effects (font (size 1.27 1.27)) hide)
+    )
+    (property "Part Number" "C0603C104M4RAC7411" (id 4) (at 349.25 92.71 0)
       (effects (font (size 1.27 1.27)) hide)
     )
@@
       (effects (font (size 1.27 1.27)) hide)
     )
+    (property "Part Number" "RNCP0603FTD10K0" (id 4) (at 190.5 138.43 0)
+      (effects (font (size 1.27 1.27)) hide)
+    )
     (pin "1")
     (pin "2")
@@
     )
     (property "Datasheet" "~" (id 3) (at 140.97 62.23 0)
+      (effects (font (size 1.27 1.27)) hide)
+    )
+    (property "Part Number" "RC0603FR-070RL" (id 4) (at 140.97 62.23 0)
       (effects (font (size 1.27 1.27)) hide)
     )
@@
       (effects (font (size 1.27 1.27)) hide)
     )
+    (property "Part Number" "RC0603JR-07300RL" (id 4) (at 40.64 106.68 0)
+      (effects (font (size 1.27 1.27)) hide)
+    )
     (pin "1")
     (pin "2")
@@
     )
     (property "Datasheet" "~" (id 3) (at 304.8 102.87 0)
+      (effects (font (size 1.27 1.27)) hide)
+    )
+    (property "Part Number" "CL10A105KA8NNNC" (id 4) (at 304.8 102.87 0)
       (effects (font (size 1.27 1.27)) hide)
     )
@@
     )
     (property "Datasheet" "~" (id 3) (at 243.84 57.15 0)
+      (effects (font (size 1.27 1.27)) hide)
+    )
+    (property "Part Number" "C0603C104M4RAC7411" (id 4) (at 243.84 57.15 0)
       (effects (font (size 1.27 1.27)) hide)
     )
@@
       (effects (font (size 1.27 1.27)) hide)
     )
+    (property "Part Number" "C0603C104M4RAC7411" (id 4) (at 252.73 92.71 0)
+      (effects (font (size 1.27 1.27)) hide)
+    )
     (pin "1")
     (pin "2")
@@
       (effects (font (size 1.27 1.27)) hide)
     )
+    (property "Part Number" "C0603C104M4RAC7411" (id 4) (at 303.53 92.71 0)
+      (effects (font (size 1.27 1.27)) hide)
+    )
     (pin "1")
     (pin "2")
@@
       (effects (font (size 1.27 1.27)) hide)
     )
+    (property "Part Number" "RC0603FR-1327RL" (id 4) (at 322.58 123.19 0)
+      (effects (font (size 1.27 1.27)) hide)
+    )
     (pin "1")
     (pin "2")
@@
     )
     (property "Datasheet" "~" (id 3) (at 217.17 165.1 0)
+      (effects (font (size 1.27 1.27)) hide)
+    )
+    (property "Part Number" "C0603C270J3GAC7867" (id 4) (at 217.17 165.1 0)
       (effects (font (size 1.27 1.27)) hide)
     )
@@
       (effects (font (size 1.27 1.27)) hide)
     )
+    (property "Part Number" "RC0603JR-07300RL" (id 4) (at 45.72 116.84 0)
+      (effects (font (size 1.27 1.27)) hide)
+    )
     (pin "1")
     (pin "2")
@@
       (effects (font (size 1.27 1.27)) hide)
     )
+    (property "Part Number" "CL10A105KA8NNNC" (id 4) (at 254 102.87 0)
+      (effects (font (size 1.27 1.27)) hide)
+    )

Commit message: Updating gerbers and adding firmware folder
Parts:
- C19, C20: Part Number CL10A105KA8NNNC -> CL10B104KA8NNNC
- U1, U2, U3, U4: Part Number AH49-E -> AH49ENTR-G1
- U5: Part Number NCP1117-3.3_SOT223 -> AZ1117IH-3.3TRG1
- U7: Part Number RP2040 -> SC0914(13)
- U8: Part Number WE-TVS-82400102 -> 82400102
Changed lines of the file:
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@@
       (effects (font (size 1.27 1.27)) hide)
     )
-    (property "Part Number" "NCP1117-3.3_SOT223" (id 4) (at 261.62 53.34 0)
+    (property "Part Number" "AZ1117IH-3.3TRG1" (id 4) (at 261.62 53.34 0)
       (effects (font (size 1.27 1.27)) hide)
     )
@@
       (effects (font (size 1.27 1.27)) hide)
     )
-    (property "Part Number" "AH49-E" (id 4) (at 107.95 50.8 0)
+    (property "Part Number" "AH49ENTR-G1" (id 4) (at 107.95 50.8 0)
       (effects (font (size 1.27 1.27)) hide)
     )
@@
       (effects (font (size 1.27 1.27)) hide)
     )
-    (property "Part Number" "AH49-E" (id 4) (at 137.16 50.8 0)
+    (property "Part Number" "AH49ENTR-G1" (id 4) (at 137.16 50.8 0)
       (effects (font (size 1.27 1.27)) hide)
     )
@@
       (effects (font (size 1.27 1.27)) hide)
     )
-    (property "Part Number" "AH49-E" (id 4) (at 50.8 50.8 0)
+    (property "Part Number" "AH49ENTR-G1" (id 4) (at 50.8 50.8 0)
       (effects (font (size 1.27 1.27)) hide)
     )
@@
       (effects (font (size 1.27 1.27)) hide)
     )
-    (property "Part Number" "RP2040" (id 4) (at 283.21 163.83 0)
+    (property "Part Number" "SC0914(13)" (id 4) (at 283.21 163.83 0)
       (effects (font (size 1.27 1.27)) hide)
     )
@@
       (effects (font (size 1.27 1.27)) hide)
     )
-    (property "Part Number" "CL10A105KA8NNNC" (id 4) (at 304.8 102.87 0)
+    (property "Part Number" "CL10B104KA8NNNC" (id 4) (at 304.8 102.87 0)
       (effects (font (size 1.27 1.27)) hide)
     )
@@
       (effects (font (size 1.27 1.27)) hide)
     )
-    (property "Part Number" "WE-TVS-82400102" (id 4) (at 81.28 189.23 0)
+    (property "Part Number" "82400102" (id 4) (at 81.28 189.23 0)
       (effects (font (size 1.27 1.27)) hide)
     )
@@
       (effects (font (size 1.27 1.27)) hide)
     )
-    (property "Part Number" "AH49-E" (id 4) (at 78.74 50.8 0)
+    (property "Part Number" "AH49ENTR-G1" (id 4) (at 78.74 50.8 0)
       (effects (font (size 1.27 1.27)) hide)
     )
@@
       (effects (font (size 1.27 1.27)) hide)
     )
-    (property "Part Number" "CL10A105KA8NNNC" (id 4) (at 254 102.87 0)
-      (effects (font (size 1.27 1.27)) hide)
-    )
+    (property "Part Number" "CL10B104KA8NNNC" (id 4) (at 254 102.87 0)
+      (effects (font (size 1.27 1.27)) hide)
+    )
